File: pcb_weegschaal/weegschaal.kicad_sch (KiCad schematic)
At the start: 29 parts, among them J1 Conn_01x04_Pin, J2 Screw_Terminal_01x03, J3 Conn_01x06_Pin, J7 Barrel_Jack, J8 Conn_01x04_Pin, K1 SANYOU_SRD_Form_C, Q1 MMBT3906, SW1 EN, SW2 FLASH, U1 ESP32-WROOM-32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

Commit message: pcb weegschaal
Parts:
- removed J2: Screw_Terminal_01x03, TerminalBlock:TerminalBlock_bornier-3_P5.08mm, symbol Connector:Screw_Terminal_01x03
- removed K1: SANYOU_SRD_Form_C, Relay_THT:Relay_SPDT_SANYOU_SRD_Series_Form_C, symbol Relay:SANYOU_SRD_Form_C
- removed Q1: MMBT3906, Package_TO_SOT_SMD:SOT-23, symbol Transistor_BJT:MMBT3906
- removed R10: 1k, Resistor_SMD:R_0805_2012Metric_Pad1.20x1.40mm_HandSolder, symbol Device:R
- added Kroonsteen1: Screw_Terminal_01x03, TerminalBlock:TerminalBlock_bornier-3_P5.08mm, symbol Connector:Screw_Terminal_01x03
- added Q1: Q_NPN_BCE, Package_TO_SOT_SMD:SOT-23, symbol Device:Q_NPN_BCE
- added Relais1: SANYOU_SRD_Form_C, Relay_THT:Relay_SPDT_SANYOU_SRD_Series_Form_C, symbol Relay:SANYOU_SRD_Form_C
- added U2: EL817, Package_DIP:DIP-4_W7.62mm, symbol Isolator:EL817
- D3: value D -> 1n4148
Connections:
- net +12V: now also Relais1.1; no longer R8.1
- net GND: now also Kroonsteen1.3 (Pin_3), Q1.3 (E); no longer D3.2 (A), R8.2, R9.2
- net GPIO32: now also U2.2
- net VDD: now also D3.1 (K), R8.1, Relais1.5, U2.4
- net at R9.1: now also U2.3; no longer D3.1 (K)
- new net: R8.2, U2.1
- new net: Kroonsteen1.1 (Pin_1), Relais1.4
- new net: Kroonsteen1.2 (Pin_2), Relais1.3
- new net: D3.2 (A), Q1.2 (C), Relais1.2
- new net: Q1.1 (B), R9.2
